File: hardware/signal_board/concept/cell.sch (KiCad schematic (older format))
At the start: 75 parts, among them Q1 Q_NMOS_GDS, Q10 Q_NMOS_GDS, Q2 Q_NMOS_GDS, Q3 Q_PMOS_GDS, Q4 Q_NMOS_GDS, Q5 Q_PMOS_GDS, Q6 Q_NMOS_GDS, Q7 Q_NMOS_GDS, Q8 Q_NMOS_GDS, Q9 Q_NMOS_GDS, U5 LM324, U6 LM324, U7 MCP6001-OT, U8 MCP6001-OT, U9 ADS1118IDGS

Commit message: Add priduction board
Parts:
- removed C35, C36, C39, C40, C41, C42, C43, C44, C53, C54: 0.1u, Capacitor_SMD:C_0603_1608Metric, symbol Device:C
- removed C37, C38, C45, C46, C47, C48, C49, C50: 100p, Capacitor_SMD:C_0603_1608Metric, symbol Device:C
- removed C51, C52: 0.22u, Capacitor_SMD:C_0603_1608Metric, symbol Device:C
- removed D5, D6: 1.25V, Package_TO_SOT_SMD:SOT-23, symbol Device:D_Zener
- removed Q1, Q2, Q7, Q8: Q_NMOS_GDS, Package_TO_SOT_SMD:SOT-23, symbol Device:Q_NMOS_GDS
- removed Q3, Q5: Q_PMOS_GDS, Package_TO_SOT_SMD:TO-252-2, symbol Device:Q_PMOS_GDS
- removed Q4, Q6: Q_NMOS_GDS, Package_TO_SOT_SMD:TO-252-2, symbol Device:Q_NMOS_GDS
- removed R10, R11, R12, R13, R18, R19, R32, R33, R34, R35: 10k, Resistor_SMD:R_0603_1608Metric, symbol Device:R
- removed R14, R15, R20, R21, R22, R23, R24, R25, R30, R31, R36, R37, R38, R39: 1k, Resistor_SMD:R_0603_1608Metric, symbol Device:R
- removed R16, R17: 100k, Resistor_SMD:R_0603_1608Metric, symbol Device:R
- removed R26, R27: 9.1k, Resistor_SMD:R_0603_1608Metric, symbol Device:R
- removed R28, R29: 1k, Resistor_SMD:R_1206_3216Metric, symbol Device:R
- removed U5, U6: LM324, Package_SO:SOIC-14_3.9x8.7mm_P1.27mm, symbol Amplifier_Operational:LM324
- removed U7, U8: MCP6001-OT, Package_TO_SOT_SMD:SOT-23-5, symbol Amplifier_Operational:MCP6001-OT
- Q1: renamed from Q9; value Q_NMOS_GDS -> Q_NMOS_GSD; symbol Device:Q_NMOS_GDS -> Device:Q_NMOS_GSD
- Q2: renamed from Q10; value Q_NMOS_GDS -> Q_NMOS_GSD; symbol Device:Q_NMOS_GDS -> Device:Q_NMOS_GSD
- renumbered C55 to C1, L2 to L1, R40 to R1, R41 to R2, R42 to R3, R43 to R4, R44 to R5, R45 to R6, U9 to U1
Connections:
- net PFC_GATE_A_HIGH: now also Q1.3 (D); no longer Q1.2 (D)
- net PFC_GATE_A_LOW: now also Q1.2 (S); no longer Q1.3 (S)
- net PFC_GATE_B_HIGH: now also Q2.3 (D); no longer Q2.2 (D)
- net PFC_GATE_B_LOW: now also Q2.2 (S); no longer Q2.3 (S)
- net CurrentSource_A_Sheet/PFC_CRNT: now reaches R1.1, U1.4 (AIN0)
- net CurrentSource_B_Sheet/PFC_CRNT: now reaches R2.1, U1.6 (AIN2)
Other:
- moved on the sheet: C38, L4, Q14, Q15, R53, R54, R55, R56, R57, R58, U10
