File: hardware/signal_board/concept/core.sch (KiCad schematic (older format))
At the start: 56 parts, among them SW1 SW_Push, SW2 SW_Push, SW3 SW_Push, SW4 SW_Push, U1 STM32F103R(F-G)Tx_u, U2 XC6SLX9-TQG144, U3 W25Q32JVSS, U4 MCP6002-xMS, Y1 8MHz

Commit message: Add priduction board
Parts:
- U20: renamed from U1; symbol stm32:STM32F103R(F-G)Tx_u -> top-rescue:STM32F103R(F-G)Tx_u-stm32
- renumbered C27 to C100, C28 to C101, C29 to C102, C30 to C103, C31 to C104, C32 to C105, C33 to C106, C34 to C107, C1 to C74, C2 to C75, C3 to C76, C4 to C77, C5 to C78, C6 to C79, C7 to C80, C8 to C81, C9 to C82, C10 to C83, C11 to C84, C12 to C85, C13 to C86, C14 to C87, C15 to C88, C16 to C89, C17 to C90, C18 to C91, C19 to C92, C20 to C93, C21 to C94, C22 to C95, C23 to C96, C24 to C97, C25 to C98, C26 to C99, D1 to D11, D2 to D12, D3 to D13, D4 to D14, R1 to R109, R2 to R110, R3 to R111, R4 to R112, R5 to R113, R6 to R114, R7 to R115, R8 to R116, R9 to R117, U2 to U21, U3 to U22, U4 to U23
Connections:
- net ADS1118_MISO: now also U20.56 (PB4/SPI1_MISO/SPI3_MISO/SYS_NJTRST/TIM3_CH1); no longer U21.2 (IO_L83P_3)
- net ADS1118_MOSI: now also U20.57 (PB5/I2C1_SMBA/I2S3_SD/SPI1_MOSI/SPI3_MOSI/TIM3_CH2); no longer U21.1 (IO_L83N_VREF_3)
- net ADS1118_SCK: now also U20.55 (PB3/I2S3_CK/SPI1_SCK/SPI3_SCK/SYS_JTDO-TRACESWO/TIM2_CH2); no longer U21.5 (IO_L52N_3)
- net W25Q32_NCS: now also U20.30 (PB11/ADC1_EXTI11/ADC2_EXTI11/I2C2_SDA/TIM2_CH4/USART3_RX); no longer U21.139 (IO_L3N_0)
- net PFC_STOP_13: now reaches U21.116 (IO_L64N_SCP4_0)
- net PFC_STOP_14: now reaches U21.117 (IO_L64P_SCP5_0)
- net PFC_STOP_15: now reaches U21.118 (IO_L63N_SCP6_0)
- net PFC_STOP_16: now reaches U21.119 (IO_L63P_SCP7_0)
- net PFC_STOP_17: now reaches U21.120 (IO_L62N_VREF_0)
- net PFC_STOP_18: now reaches U21.121 (IO_L62P_0)
- net PFC_STOP_19: now reaches U21.126 (IO_L36N_GCLK14_0)
- net PFC_STOP_20: now reaches U21.127 (IO_L36P_GCLK15_0)
- net PFC_STOP_21: now reaches U21.133 (IO_L34N_GCLK18_0)
- net PFC_STOP_9: now reaches U21.74 (IO_L74N_DOUT_BUSY_1)
- net PFC_STOP_10: now reaches U21.75 (IO_L74P_AWAKE_1)
- net PFC_STOP_11: now reaches U21.87 (IO_L42N_GCLK6_TRDY1_1)
- net PFC_STOP_12: now reaches U21.88 (IO_L42P_GCLK7_1)
- net PFC_STOP_0: now reaches U21.16 (IO_L43N_GCLK22_IRDY2_3)
- net PFC_STOP_1: now reaches U21.17 (IO_L43P_GCLK23_3)
- net PFC_STOP_2: now reaches U21.38 (IO_L65N_CSO_B_2)
- net PFC_STOP_3: now reaches U21.57 (IO_L14N_D12_2)
- net PFC_STOP_4: now reaches U21.58 (IO_L14P_D11_2)
- net PFC_STOP_5: now reaches U21.59 (IO_L13N_D10_2)
- net PFC_STOP_6: now reaches U21.61 (IO_L12N_D2_MISO3_2)
- net PFC_STOP_7: now reaches U21.66 (IO_L2N_CMPMOSI_2)
- net PFC_STOP_8: now reaches U21.67 (IO_L2P_CMPCLK_2)
- net ADS1118_NSC_0 renamed ADS1118_NCS_0
- net ADS1118_NSC_1 renamed ADS1118_NCS_1
- net ADS1118_NSC_10 renamed ADS1118_NCS_10
- net ADS1118_NSC_11 renamed ADS1118_NCS_11
- net ADS1118_NSC_12 renamed ADS1118_NCS_12
- net ADS1118_NSC_13 renamed ADS1118_NCS_13
- net ADS1118_NSC_14 renamed ADS1118_NCS_14
- net ADS1118_NSC_2 renamed ADS1118_NCS_2
- net ADS1118_NSC_3 renamed ADS1118_NCS_3
- net ADS1118_NSC_4 renamed ADS1118_NCS_4
- net ADS1118_NSC_5 renamed ADS1118_NCS_5
- net ADS1118_NSC_6 renamed ADS1118_NCS_6
- net ADS1118_NSC_7 renamed ADS1118_NCS_7
- net ADS1118_NSC_8 renamed ADS1118_NCS_8
- net ADS1118_NSC_9 renamed ADS1118_NCS_9
- net W25Q32_MISO renamed PFC_STOP_23
- net PFC_STOP_23: no longer U22.2 (DO(IO1))
- net W25Q32_MOSI renamed PFC_STOP_22
- net PFC_STOP_22: no longer U22.5 (DI(IO0))
- net W25Q32_SCK renamed PFC_STOP_24
- net PFC_STOP_24: no longer U22.6 (CLK)
- net XC6SLX9_MISO renamed XC6SLX9_W25Q32_MISO
- net XC6SLX9_W25Q32_MISO: now also U22.2 (DO(IO1))
- net XC6SLX9_MOSI renamed XC6SLX9_W25Q32_MOSI
- net XC6SLX9_W25Q32_MOSI: now also U22.5 (DI(IO0))
- net XC6SLX9_ROUTABLE_MISO renamed PFC_STOP_27
- net PFC_STOP_27: no longer U20.56 (PB4/SPI1_MISO/SPI3_MISO/SYS_NJTRST/TIM3_CH1)
- net XC6SLX9_ROUTABLE_MOSI renamed PFC_STOP_26
- net PFC_STOP_26: no longer U20.57 (PB5/I2C1_SMBA/I2S3_SD/SPI1_MOSI/SPI3_MOSI/TIM3_CH2)
- net XC6SLX9_ROUTABLE_NCS: no longer names the net of U20.50 (PA15/ADC1_EXTI15/ADC2_EXTI15/I2S3_WS/SPI1_NSS/SPI3_NSS/SYS_JTDI/TIM2_CH1/TIM2_ETR)
- net XC6SLX9_ROUTABLE_NCS: no longer U21.143 (IO_L1N_VREF_0)
- net XC6SLX9_ROUTABLE_SCK renamed PFC_STOP_28
- net PFC_STOP_28: no longer U20.55 (PB3/I2S3_CK/SPI1_SCK/SPI3_SCK/SYS_JTDO-TRACESWO/TIM2_CH2)
- net XC6SLX9_SCK renamed XC6SLX9_W25Q32_SCK
- net XC6SLX9_W25Q32_SCK: now also U22.6 (CLK)
- new net PFC_STOP_25: U21.139 (IO_L3N_0)
- new net PFC_STOP_29: U21.143 (IO_L1N_VREF_0)
- no-connect marks 45 -> 26
Other:
- moved on the sheet: C76, C77, C79, C80, C82, C83, C85, C86, C88, C89, U21C, U21D
