File: hardware/signal_board/concept/ports.sch (KiCad schematic (older format))
At the start: 5 parts, among them J1 Conn_01x04, J2 USB_OTG, J3 Conn_01x02, J4 Barrel_Jack_Switch

Commit message: Add priduction board
Parts:
- renumbered J4 to J3, J3 to J4, R109 to R108
Changed lines of the file:
@@
 $Descr A4 11693 8268
 encoding utf-8
-Sheet 12 12
+Sheet 15 16
 Title ""
 Date ""
@@
 P 1700 2400
 AR Path="/63DEFF92/5E56786B" Ref="#PWR?"  Part="1"
-AR Path="/5E56622A/5E56786B" Ref="#PWR085"  Part="1"
-F 0 "#PWR085" H 1700 2150 50  0001 C CNN
+AR Path="/5E56622A/5E56786B" Ref="#PWR078"  Part="1"
+F 0 "#PWR078" H 1700 2150 50  0001 C CNN
 F 1 "GNDD" H 1704 2245 50  0000 C CNN
 F 2 "" H 1700 2400 50  0001 C CNN
@@
 P 1900 2350
 AR Path="/63DEFF92/5E567873" Ref="R?"  Part="1"
-AR Path="/5E56622A/5E567873" Ref="R109"  Part="1"
-F 0 "R109" V 1800 2350 50  0000 C CNN
+AR Path="/5E56622A/5E567873" Ref="R108"  Part="1"
+F 0 "R108" V 1800 2350 50  0000 C CNN
 F 1 "1k" V 1900 2350 50  0000 C CNN
 F 2 "Resistor_SMD:R_0603_1608Metric" V 1830 2350 50  0001 C CNN
@@
 P 2050 1450
 AR Path="/63DEFF92/5E567884" Ref="J?"  Part="1"
-AR Path="/5E56622A/5E567884" Ref="J3"  Part="1"
-F 0 "J3" V 2014 1262 50  0000 R CNN
+AR Path="/5E56622A/5E567884" Ref="J4"  Part="1"
+F 0 "J4" V 2014 1262 50  0000 R CNN
 F 1 "Conn_01x02" V 1923 1262 50  0000 R CNN
 F 2 "Connector_PinHeader_2.54mm:PinHeader_1x02_P2.54mm_Vertical" H 2050 1450 50  0001 C CNN
@@
 P 1800 3250
 AR Path="/63DEFF92/5E57E355" Ref="#PWR?"  Part="1"
-AR Path="/5E56622A/5E57E355" Ref="#PWR086"  Part="1"
-F 0 "#PWR086" H 1800 3000 50  0001 C CNN
+AR Path="/5E56622A/5E57E355" Ref="#PWR079"  Part="1"
+F 0 "#PWR079" H 1800 3000 50  0001 C CNN
 F 1 "GNDD" H 1804 3095 50  0000 C CNN
 F 2 "" H 1800 3250 50  0001 C CNN
@@
 P 3850 2050
 AR Path="/63DEFF92/5E58099C" Ref="#PWR?"  Part="1"
-AR Path="/5E56622A/5E58099C" Ref="#PWR087"  Part="1"
-F 0 "#PWR087" H 3850 1800 50  0001 C CNN
+AR Path="/5E56622A/5E58099C" Ref="#PWR081"  Part="1"
+F 0 "#PWR081" H 3850 1800 50  0001 C CNN
 F 1 "GNDD" V 3850 1850 50  0000 C CNN
 F 2 "" H 3850 2050 50  0001 C CNN
@@
 	3850 2050 4350 2050
 $Comp
-L Connector:Barrel_Jack_Switch J4
+L Connector:Barrel_Jack_Switch J3
 U 1 1 5F341D99
 P 1700 3850
-F 0 "J4" H 1757 4167 50  0000 C CNN
+F 0 "J3" H 1757 4167 50  0000 C CNN
 F 1 "Barrel_Jack_Switch" H 1757 4076 50  0000 C CNN
 F 2 "Connector_BarrelJack:BarrelJack_Horizontal" H 1750 3810 50  0001 C CNN
@@
 VCC12V
 $Comp
-L power:GNDPWR #PWR0101
+L power:GNDPWR #PWR080
 U 1 1 5F345610
 P 2050 4000
-F 0 "#PWR0101" H 2050 3800 50  0001 C CNN
+F 0 "#PWR080" H 2050 3800 50  0001 C CNN
 F 1 "GNDPWR" H 2054 3846 50  0000 C CNN
 F 2 "" H 2050 3950 50  0001 C CNN
@@
 VCC12V
 $Comp
-L power:GNDPWR #PWR0102
+L power:GNDPWR #PWR082
 U 1 1 5F349B76
 P 3950 2150
-F 0 "#PWR0102" H 3950 1950 50  0001 C CNN
+F 0 "#PWR082" H 3950 1950 50  0001 C CNN
 F 1 "GNDPWR" V 3954 2041 50  0000 R CNN
 F 2 "" H 3950 2100 50  0001 C CNN
