File: hardware/signal_board/concept/power.sch (KiCad schematic (older format))
At the start: 37 parts, among them Q11 Q_NMOS_GDS, U10 L5973D, U11 LM3488MM, U12 AMS1117-3.3, U13 AMS1117

Commit message: Add priduction board
Parts:
- D4: renamed from D8; footprint Package_TO_SOT_SMD:TO-252-2 -> Diode_SMD:D_SMC
- renumbered C56 to C22, C57 to C23, C58 to C24, C59 to C25, C60 to C26, C61 to C27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
