File: hardware/signal_board/production/core.sch (KiCad schematic (older format))
At the start: 56 parts, among them SW1 SW_Push, SW2 SW_Push, SW3 SW_Push, SW4 SW_Push, U20 STM32F103R(F-G)Tx_u, U21 XC6SLX9-TQG144, U22 W25Q32JVSS, U23 MCP6002-xMS, Y1 8MHz

Commit message: fix
Parts:
- added R630: 9.1k, Resistor_SMD:R_0603_1608Metric, symbol Device:R
- added R631, R632, R633: 1k, Resistor_SMD:R_0603_1608Metric, symbol Device:R
Connections:
- net GNDD: now also R631.2, R633.2
- net U_PFC_FB_OVP_ADJ: now also U20.22 (PA6/ADC1_IN6/ADC2_IN6/SPI1_MISO/TIM13_CH1/TIM1_BKIN/TIM3_CH1/TIM8_BKIN)
- net U_PFC_VCC_ADJ: now also U20.23 (PA7/ADC1_IN7/ADC2_IN7/SPI1_MOSI/TIM14_CH1/TIM1_CH1N/TIM3_CH2/TIM8_CH1N)
- net VBUS_ADC: now reaches U20.16 (PA2/ADC1_IN2/ADC2_IN2/ADC3_IN2/TIM2_CH3/TIM5_CH3/TIM9_CH1/USART2_TX)
- net VBUS_ADC: now also R630.2, R631.1
- net V_FB_OVP_ADC: now reaches U20.17 (PA3/ADC1_IN3/ADC2_IN3/ADC3_IN3/TIM2_CH4/TIM5_CH4/TIM9_CH2/USART2_RX)
- net V_FB_OVP_ADC: now also R632.2, R633.1
- new net VCC30V: R630.1
- new net V_FB_OVP: R632.1
- no-connect marks 26 -> 22
Changed lines of the file:
@@
 	0    -1   -1   0
 $EndComp
-Wire Wire Line
-	6600 3850 7600 3850
-Wire Wire Line
-	6600 3750 7600 3750
 Text Label 7600 3750 2    50   ~ 0
 U_PFC_FB_OVP_ADJ_DAC
@@
 VDD1.25V
 Wire Wire Line
+	11500 17050 10650 17050
+Wire Wire Line
 	11500 16950 10650 16950
-Wire Wire Line
-	11500 16850 10650 16850
-Text Label 10650 16850 0    50   ~ 0
+Text Label 10650 16950 0    50   ~ 0
 U_PFC_FB_OVP_ADJ
-Text Label 10650 16950 0    50   ~ 0
+Text Label 10650 17050 0    50   ~ 0
 U_PFC_VCC_ADJ
-Text HLabel 11500 16850 2    50   Output ~ 0
+Text HLabel 11500 16950 2    50   Output ~ 0
 U_PFC_FB_OVP_ADJ
-Text HLabel 11500 16950 2    50   Output ~ 0
+Text HLabel 11500 17050 2    50   Output ~ 0
 U_PFC_VCC_ADJ
 Text Label 7600 7300 2    50   ~ 0
@@
 NoConn ~ 6600 3350
 NoConn ~ 6600 3450
-NoConn ~ 6600 3550
-NoConn ~ 6600 3650
-NoConn ~ 6600 3950
-NoConn ~ 6600 4050
 NoConn ~ 6600 5300
 NoConn ~ 6600 5400
@@
 Connection ~ 12400 9650
 Wire Wire Line
-	11500 17150 10650 17150
-Wire Wire Line
 	11500 17250 10650 17250
-Text Label 10650 17150 0    50   ~ 0
+Wire Wire Line
+	11500 17350 10650 17350
+Text Label 10650 17250 0    50   ~ 0
 STM32F103_USB_D-
-Text Label 10650 17250 0    50   ~ 0
+Text Label 10650 17350 0    50   ~ 0
 STM32F103_USB_D+
 Wire Wire Line
-	11500 17450 10650 17450
-Text Label 10650 17450 0    50   ~ 0
+	11500 17550 10650 17550
+Text Label 10650 17550 0    50   ~ 0
 STM32F103_SWDIO
-Text Label 10650 17550 0    50   ~ 0
+Text Label 10650 17650 0    50   ~ 0
 STM32F103_SWCLK
 Wire Wire Line
-	10650 17550 11500 17550
-Text HLabel 11500 17150 2    50   BiDi ~ 0
+	10650 17650 11500 17650
+Text HLabel 11500 17250 2    50   BiDi ~ 0
 STM32F103_USB_D-
-Text HLabel 11500 17250 2    50   BiDi ~ 0
+Text HLabel 11500 17350 2    50   BiDi ~ 0
 STM32F103_USB_D+
-Text HLabel 11500 17450 2    50   BiDi ~ 0
+Text HLabel 11500 17550 2    50   BiDi ~ 0
 STM32F103_SWDIO
-Text HLabel 11500 17550 2    50   BiDi ~ 0
+Text HLabel 11500 17650 2    50   BiDi ~ 0
 STM32F103_SWCLK
 Wire Wire Line
@@
 	1750 11750 2750 11750
 Wire Wire Line
+	6600 3850 7600 3850
+Wire Wire Line
+	6600 3750 7600 3750
+Wire Wire Line
+	6600 3950 7600 3950
+Wire Wire Line
+	6600 4050 7600 4050
+Text Label 7600 3950 2    50   ~ 0
+U_PFC_FB_OVP_ADJ
+Text Label 7600 4050 2    50   ~ 0
+U_PFC_VCC_ADJ
+$Comp
+L Device:R R630
+U 1 1 5E7C0E62
+P 8700 6800
+F 0 "R630" H 8770 6846 50  0000 L CNN
+F 1 "9.1k" H 8770 6755 50  0000 L CNN
+F 2 "Resistor_SMD:R_0603_1608Metric" V 8630 6800 50  0001 C CNN
+F 3 "~" H 8700 6800 50  0001 C CNN
+	1    8700 6800
+	1    0    0    -1
+$EndComp
+$Comp
+L Device:R R631
+U 1 1 5E7C16DE
+P 8700 7200
+F 0 "R631" H 8770 7246 50  0000 L CNN
+F 1 "1k" H 8770 7155 50  0000 L CNN
+F 2 "Resistor_SMD:R_0603_1608Metric" V 8630 7200 50  0001 C CNN
+F 3 "~" H 8700 7200 50  0001 C CNN
+	1    8700 7200
+	1    0    0    -1
+$EndComp
+$Comp
+L power:GNDD #PWR070
+U 1 1 5E7C1A7D
+P 8700 7350
+F 0 "#PWR070" H 8700 7100 50  0001 C CNN
+F 1 "GNDD" H 8704 7195 50  0000 C CNN
+F 2 "" H 8700 7350 50  0001 C CNN
+F 3 "" H 8700 7350 50  0001 C CNN
+	1    8700 7350
+	1    0    0    -1
+$EndComp
+Wire Wire Line
+	8700 6950 8700 7000
+Wire Wire Line
+	8700 6650 8700 6600
+Wire Wire Line
+	8700 6600 9000 6600
+Text Label 9000 6600 2    50   ~ 0
+VCC30V
+Wire Wire Line
+	8700 7000 8250 7000
+Connection ~ 8700 7000
+Wire Wire Line
+	8700 7000 8700 7050
+Text Label 8250 7000 0    50   ~ 0
+VBUS_ADC
+Text Label 10650 15200 0    50   ~ 0
+VCC30V
+Wire Wire Line
+	10650 15200 11450 15200
+Text HLabel 11450 15200 2    50   Input ~ 0
+VCC30V
+Wire Wire Line
+	6600 3550 7600 3550
+Text Label 7600 3550 2    50   ~ 0
+VBUS_ADC
+$Comp
+L Device:R R632
+U 1 1 5EADD700
+P 8700 7900
+F 0 "R632" H 8770 7946 50  0000 L CNN
+F 1 "1k" H 8770 7855 50  0000 L CNN
+F 2 "Resistor_SMD:R_0603_1608Metric" V 8630 7900 50  0001 C CNN
+F 3 "~" H 8700 7900 50  0001 C CNN
+	1    8700 7900
+	1    0    0    -1
+$EndComp
+$Comp
+L Device:R R633
+U 1 1 5EADD706
+P 8700 8300
+F 0 "R633" H 8770 8346 50  0000 L CNN
+F 1 "1k" H 8770 8255 50  0000 L CNN
+F 2 "Resistor_SMD:R_0603_1608Metric" V 8630 8300 50  0001 C CNN
+F 3 "~" H 8700 8300 50  0001 C CNN
+	1    8700 8300
+	1    0    0    -1
+$EndComp
+$Comp
+L power:GNDD #PWR071
+U 1 1 5EADD70C
+P 8700 8450
+F 0 "#PWR071" H 8700 8200 50  0001 C CNN
+F 1 "GNDD" H 8704 8295 50  0000 C CNN
+F 2 "" H 8700 8450 50  0001 C CNN
+F 3 "" H 8700 8450 50  0001 C CNN
+	1    8700 8450
+	1    0    0    -1
+$EndComp
+Wire Wire Line
+	8700 8050 8700 8100
+Wire Wire Line
+	8700 7750 8700 7700
+Wire Wire Line
+	8700 7700 9050 7700
+Text Label 9050 7700 2    50   ~ 0
+V_FB_OVP
+Wire Wire Line
+	8700 8100 8100 8100
+Connection ~ 8700 8100
+Wire Wire Line
+	8700 8100 8700 8150
+Text Label 8100 8100 0    50   ~ 0
+V_FB_OVP_ADC
+Text Label 7600 3650 2    50   ~ 0
+V_FB_OVP_ADC
+Wire Wire Line
+	6600 3650 7600 3650
+Text Label 10650 16850 0    50   ~ 0
+V_FB_OVP
+Wire Wire Line
+	10650 16850 11500 16850
+Text HLabel 11500 16850 2    50   Input ~ 0
+V_FB_OVP
+Wire Wire Line
 	1550 11950 2750 11950
